File: Power.sch (KiCad schematic (older format))
At the start: 13 parts, among them P1 CONN_12X2, SW1 SWITCH_INV

Commit message: Am Ende der 5. Woche.
Parts:
- L1, L2, L3: value INDUCTOR -> CM322522-220KL; MFG Name (none) -> Bournes
- P1: value CONN_12X2 -> 24 Pin MiniFit JR; MFG Name (none) -> Molex; MFG Part Number (none) -> 39-30-1240
- SW1: value SWITCH_INV -> PowerSwitch; MFG Name (none) -> C&K Components; MFG Part Number (none) -> =s102011MA1QN1
- TH1, TH2, TH3, TH4: value THERMISTOR -> MINISMDC050F-2; MFG Name (none) -> TE Connectivity; MFG Part Number (none) -> MINISMDC050F-2
Changed lines of the file:
@@
 Sheet 4 9
 Title ""
-Date "17 feb 2014"
+Date "22 feb 2014"
 Rev ""
 Comp ""
@@
 P 2600 2500
 F 0 "P1" H 2600 3150 60  0000 C CNN
-F 1 "CONN_12X2" V 2600 2500 50  0000 C CNN
+F 1 "24 Pin MiniFit JR" V 2600 2500 50  0000 C CNN
 F 2 "" H 2600 2500 60  0000 C CNN
 F 3 "" H 2600 2500 60  0000 C CNN
+F 4 "Molex" H 2600 2500 60  0001 C CNN "MFG Name"
+F 5 "39-30-1240" H 2600 2500 60  0001 C CNN "MFG Part Number"
 	1    2600 2500
 	1    0    0    -1
 $EndComp
 $Comp
-L GND #PWR13
+L GND #PWR020
 U 1 1 52F104F8
 P 1350 2200
-F 0 "#PWR13" H 1350 2200 30  0001 C CNN
+F 0 "#PWR020" H 1350 2200 30  0001 C CNN
 F 1 "GND" H 1350 2130 30  0001 C CNN
 F 2 "" H 1350 2200 60  0000 C CNN
@@
 P 4000 3600
 F 0 "SW1" H 3800 3750 50  0000 C CNN
-F 1 "SWITCH_INV" H 3850 3450 50  0000 C CNN
+F 1 "PowerSwitch" H 3850 3450 50  0000 C CNN
 F 2 "~" H 4000 3600 60  0000 C CNN
 F 3 "~" H 4000 3600 60  0000 C CNN
+F 4 "C&K Components" H 4000 3600 60  0001 C CNN "MFG Name"
+F 5 "=s102011MA1QN1" H 4000 3600 60  0001 C CNN "MFG Part Number"
 	1    4000 3600
 	1    0    0    -1
@@
 Wire Wire Line
 	3150 1950 3000 1950
-Wire Wire Line
-	3000 2150 3700 2150
 Wire Wire Line
 	3000 2050 3250 2050
@@
 	4700 3700 4700 3900
 $Comp
-L GND #PWR17
+L GND #PWR021
 U 1 1 52F10B9A
 P 4700 3900
-F 0 "#PWR17" H 4700 3900 30  0001 C CNN
+F 0 "#PWR021" H 4700 3900 30  0001 C CNN
 F 1 "GND" H 4700 3830 30  0001 C CNN
 F 2 "" H 4700 3900 60  0000 C CNN
@@
 	5450 3500 5450 3100
 $Comp
-L +3,3V #PWR20
+L +3,3V #PWR022
 U 1 1 52F10BEB
 P 5450 3100
-F 0 "#PWR20" H 5450 3060 30  0001 C CNN
+F 0 "#PWR022" H 5450 3060 30  0001 C CNN
 F 1 "+3,3V" H 5450 3210 30  0000 C CNN
 F 2 "" H 5450 3100 60  0000 C CNN
@@
 $EndComp
 $Comp
-L +12P #PWR18
+L +12P #PWR023
 U 1 1 52F10BF8
 P 4850 1500
-F 0 "#PWR18" H 4850 1470 30  0001 C CNN
+F 0 "#PWR023" H 4850 1470 30  0001 C CNN
 F 1 "+12P" H 4850 1600 30  0000 C CNN
 F 2 "" H 4850 1500 60  0000 C CNN
@@
 	4850 1500 4850 2350
 $Comp
-L -12P #PWR19
+L -12P #PWR024
 U 1 1 52F10C29
 P 5400 1500
-F 0 "#PWR19" H 5400 1630 20  0001 C CNN
+F 0 "#PWR024" H 5400 1630 20  0001 C CNN
 F 1 "-12P" H 5400 1600 30  0000 C CNN
 F 2 "" H 5400 1500 60  0000 C CNN
@@
 Wire Wire Line
 	3600 1950 3750 1950
-$Comp
-L INDUCTOR L2
-U 1 1 52F10CC6
-P 7050 2750
-F 0 "L2" V 7000 2750 40  0000 C CNN
-F 1 "INDUCTOR" V 7150 2750 40  0000 C CNN
-F 2 "~" H 7050 2750 60  0000 C CNN
-F 3 "~" H 7050 2750 60  0000 C CNN
-	1    7050 2750
-	0    -1   -1   0
-$EndComp
-$Comp
-L INDUCTOR L3
-U 1 1 52F10CD3
-P 7100 4000
-F 0 "L3" V 7050 4000 40  0000 C CNN
-F 1 "INDUCTOR" V 7200 4000 40  0000 C CNN
-F 2 "~" H 7100 4000 60  0000 C CNN
-F 3 "~" H 7100 4000 60  0000 C CNN
-	1    7100 4000
-	0    -1   -1   0
-$EndComp
 $Comp
 L C C2
@@
 $EndComp
 $Comp
-L +12P #PWR22
+L +12P #PWR025
 U 1 1 52F10D27
 P 6400 2500
-F 0 "#PWR22" H 6400 2470 30  0001 C CNN
+F 0 "#PWR025" H 6400 2470 30  0001 C CNN
 F 1 "+12P" H 6400 2600 30  0000 C CNN
 F 2 "" H 6400 2500 60  0000 C CNN
@@
 	6500 4000 6500 4250
 $Comp
-L -12P #PWR23
+L -12P #PWR026
 U 1 1 52F10DDD
 P 6500 4250
-F 0 "#PWR23" H 6500 4380 20  0001 C CNN
+F 0 "#PWR026" H 6500 4380 20  0001 C CNN
 F 1 "-12P" H 6500 4350 30  0000 C CNN
 F 2 "" H 6500 4250 60  0000 C CNN
@@
 $EndComp
 $Comp
-L GND #PWR24
+L GND #PWR027
 U 1 1 52F10DEC
 P 7300 3500
-F 0 "#PWR24" H 7300 3500 30  0001 C CNN
+F 0 "#PWR027" H 7300 3500 30  0001 C CNN
 F 1 "GND" H 7300 3430 30  0001 C CNN
 F 2 "" H 7300 3500 60  0000 C CNN
@@
 Connection ~ 7800 3350
 $Comp
-L -12V #PWR28
+L -12V #PWR028
 U 1 1 52F10E22
 P 8650 4250
-F 0 "#PWR28" H 8650 4380 20  0001 C CNN
+F 0 "#PWR028" H 8650 4380 20  0001 C CNN
 F 1 "-12V" H 8650 4350 30  0000 C CNN
 F 2 "" H 8650 4250 60  0000 C CNN
@@
 Connection ~ 7800 4000
 $Comp
-L +12V #PWR27
+L +12V #PWR029
 U 1 1 52F10E65
 P 8650 2500
-F 0 "#PWR27" H 8650 2450 20  0001 C CNN
+F 0 "#PWR029" H 8650 2450 20  0001 C CNN
 F 1 "+12V" H 8650 2600 30  0000 C CNN
 F 2 "" H 8650 2500 60  0000 C CNN
@@
 Connection ~ 7800 2750
 $Comp
-L +12C #PWR14
+L +12C #PWR030
 U 1 1 52F3B02A
 P 3050 1500
-F 0 "#PWR14" H 3050 1470 30  0001 C CNN
+F 0 "#PWR030" H 3050 1470 30  0001 C CNN
 F 1 "+12C" H 3050 1610 40  0000 C CNN
 F 2 "" H 3050 1500 60  0000 C CNN
@@
 P 3350 1950
 F 0 "TH1" V 3450 2000 50  0000 C CNN
-F 1 "THERMISTOR" V 3250 1950 50  0000 C CNN
+F 1 "MINISMDC050F-2" V 3250 1950 50  0000 C CNN
 F 2 "~" H 3350 1950 60  0000 C CNN
 F 3 "~" H 3350 1950 60  0000 C CNN
+F 4 "TE Connectivity" H 3350 1950 60  0001 C CNN "MFG Name"
+F 5 "MINISMDC050F-2" H 3350 1950 60  0001 C CNN "MFG Part Number"
 	1    3350 1950
 	0    -1   -1   0
 $EndComp
 $Comp
-L THERMISTOR TH2
-U 1 1 52F3B37D
-P 3900 2150
-F 0 "TH2" V 4000 2200 50  0000 C CNN
-F 1 "THERMISTOR" V 3800 2150 50  0000 C CNN
-F 2 "~" H 3900 2150 60  0000 C CNN
-F 3 "~" H 3900 2150 60  0000 C CNN
-	1    3900 2150
-	0    -1   -1   0
-$EndComp
-$Comp
-L THERMISTOR TH3
-U 1 1 52F3B383
-P 4500 2350
-F 0 "TH3" V 4600 2400 50  0000 C CNN
-F 1 "THERMISTOR" V 4400 2350 50  0000 C CNN
-F 2 "~" H 4500 2350 60  0000 C CNN
-F 3 "~" H 4500 2350 60  0000 C CNN
-	1    4500 2350
-	0    -1   -1   0
-$EndComp
-$Comp
-L THERMISTOR TH4
-U 1 1 52F3B389
-P 5050 2550
-F 0 "TH4" V 5150 2600 50  0000 C CNN
-F 1 "THERMISTOR" V 4950 2550 50  0000 C CNN
-F 2 "~" H 5050 2550 60  0000 C CNN
-F 3 "~" H 5050 2550 60  0000 C CNN
-	1    5050 2550
-	0    -1   -1   0
-$EndComp
-$Comp
-L +5P #PWR16
+L +5P #PWR23
 U 1 1 52FDF0C0
 P 4300 1500
-F 0 "#PWR16" H 4300 1630 20  0001 C CNN
+F 0 "#PWR23" H 4300 1630 20  0001 C CNN
 F 1 "+5P" H 4300 1600 30  0000 C CNN
 F 2 "" H 4300 1500 60  0000 C CNN
@@
 $EndComp
 $Comp
-L +3.3VP #PWR15
+L +3.3VP #PWR031
 U 1 1 52FDF0CF
 P 3750 1500
-F 0 "#PWR15" H 3800 1530 20  0001 C CNN
+F 0 "#PWR031" H 3800 1530 20  0001 C CNN
 F 1 "+3.3VP" H 3750 1590 30  0000 C CNN
 F 2 "" H 3750 1500 60  0000 C CNN
@@
 P 7000 1200
 F 0 "L1" V 6950 1200 40  0000 C CNN
-F 1 "INDUCTOR" V 7100 1200 40  0000 C CNN
+F 1 "CM322522-220KL" V 7100 1200 40  0000 C CNN
 F 2 "~" H 7000 1200 60  0000 C CNN
 F 3 "~" H 7000 1200 60  0000 C CNN
+F 4 "Bournes" H 7000 1200 60  0001 C CNN "MFG Name"
 	1    7000 1200
 	0    -1   -1   0
@@
 	7750 1200 7750 1300
 $Comp
-L GND #PWR25
+L GND #PWR032
 U 1 1 52FDF0F9
 P 7750 1900
-F 0 "#PWR25" H 7750 1900 30  0001 C CNN
+F 0 "#PWR032" H 7750 1900 30  0001 C CNN
 F 1 "GND" H 7750 1830 30  0001 C CNN
 F 2 "" H 7750 1900 60  0000 C CNN
@@
 Connection ~ 7750 1200
 $Comp
-L +5P #PWR21
+L +5P #PWR28
 U 1 1 52FDF142
 P 6350 950
-F 0 "#PWR21" H 6350 1080 20  0001 C CNN
+F 0 "#PWR28" H 6350 1080 20  0001 C CNN
 F 1 "+5P" H 6350 1050 30  0000 C CNN
 F 2 "" H 6350 950 60  0000 C CNN
@@
 $EndComp
 $Comp
-L +5V #PWR26
+L +5V #PWR033
 U 1 1 52FDF14A
 P 8600 950
-F 0 "#PWR26" H 8600 1040 20  0001 C CNN
+F 0 "#PWR033" H 8600 1040 20  0001 C CNN
 F 1 "+5V" H 8600 1040 30  0000 C CNN
 F 2 "" H 8600 950 60  0000 C CNN
@@
 Wire Wire Line
 	7750 1700 7750 1900
+$Comp
+L THERMISTOR TH2
+U 1 1 53062D4C
+P 3900 2150
+F 0 "TH2" V 4000 2200 50  0000 C CNN
+F 1 "MINISMDC050F-2" V 3800 2150 50  0000 C CNN
+F 2 "~" H 3900 2150 60  0000 C CNN
+F 3 "~" H 3900 2150 60  0000 C CNN
+F 4 "TE Connectivity" H 3900 2150 60  0001 C CNN "MFG Name"
+F 5 "MINISMDC050F-2" H 3900 2150 60  0001 C CNN "MFG Part Number"
+	1    3900 2150
+	0    -1   -1   0
+$EndComp
+$Comp
+L THERMISTOR TH3
+U 1 1 53062D54
+P 4500 2350
+F 0 "TH3" V 4600 2400 50  0000 C CNN
+F 1 "MINISMDC050F-2" V 4400 2350 50  0000 C CNN
+F 2 "~" H 4500 2350 60  0000 C CNN
+F 3 "~" H 4500 2350 60  0000 C CNN
+F 4 "TE Connectivity" H 4500 2350 60  0001 C CNN "MFG Name"
+F 5 "MINISMDC050F-2" H 4500 2350 60  0001 C CNN "MFG Part Number"
+	1    4500 2350
+	0    -1   -1   0
+$EndComp
+$Comp
+L THERMISTOR TH4
+U 1 1 53062D5C
+P 5050 2550
+F 0 "TH4" V 5150 2600 50  0000 C CNN
+F 1 "MINISMDC050F-2" V 4950 2550 50  0000 C CNN
+F 2 "~" H 5050 2550 60  0000 C CNN
+F 3 "~" H 5050 2550 60  0000 C CNN
+F 4 "TE Connectivity" H 5050 2550 60  0001 C CNN "MFG Name"
+F 5 "MINISMDC050F-2" H 5050 2550 60  0001 C CNN "MFG Part Number"
+	1    5050 2550
+	0    -1   -1   0
+$EndComp
+Wire Wire Line
+	3000 2150 3650 2150
+$Comp
+L INDUCTOR L3
+U 1 1 53062DC6
+P 7050 2750
+F 0 "L3" V 7000 2750 40  0000 C CNN
+F 1 "CM322522-220KL" V 7150 2750 40  0000 C CNN
+F 2 "~" H 7050 2750 60  0000 C CNN
+F 3 "~" H 7050 2750 60  0000 C CNN
+F 4 "Bournes" H 7050 2750 60  0001 C CNN "MFG Name"
+	1    7050 2750
+	0    -1   -1   0
+$EndComp
+$Comp
+L INDUCTOR L2
+U 1 1 53062DD9
+P 7100 4000
+F 0 "L2" V 7050 4000 40  0000 C CNN
+F 1 "CM322522-220KL" V 7200 4000 40  0000 C CNN
+F 2 "~" H 7100 4000 60  0000 C CNN
+F 3 "~" H 7100 4000 60  0000 C CNN
+F 4 "Bournes" H 7100 4000 60  0001 C CNN "MFG Name"
+	1    7100 4000
+	0    -1   -1   0
+$EndComp
 $EndSCHEMATC
