File: PowerAdjustmentMonitor.sch (KiCad schematic (older format))
At the start: 19 parts

Commit message: Am Ende der 4. Woche
Parts:
- removed R? (x2): R, ~, symbol R
- removed U? (x2): LM324, symbol LM324
Connections:
- net labels removed: V+_CURR_MON, V-_CURR_MON
- wire segments 79 -> 61
Changed lines of the file:
@@
 $Descr A4 11693 8268
 encoding utf-8
-Sheet 9 9
+Sheet 8 9
 Title ""
-Date "7 feb 2014"
+Date "14 feb 2014"
 Rev ""
 Comp ""
@@
 Connection ~ 5550 6450
 Connection ~ 5600 900
-Text HLabel 10250 6350 2    60   Output ~ 0
-V-_CURR_MON
-Text HLabel 10250 5000 2    60   Output ~ 0
-V+_CURR_MON
 $Comp
 L R R?
@@
 Wire Wire Line
 	9800 3150 9800 2650
-$Comp
-L R R?
-U 1 1 52F13CA0
-P 6100 900
-F 0 "R?" V 6180 900 40  0000 C CNN
-F 1 "R" V 6107 901 40  0000 C CNN
-F 2 "~" V 6030 900 30  0000 C CNN
-F 3 "~" H 6100 900 30  0000 C CNN
-	1    6100 900
-	0    1    -1   0
-$EndComp
-Wire Wire Line
-	5350 900  5850 900
-Wire Wire Line
-	6350 900  6700 900
 Connection ~ 6650 900
-$Comp
-L R R?
-U 1 1 52F13E0F
-P 6050 6450
-F 0 "R?" V 6130 6450 40  0000 C CNN
-F 1 "R" V 6057 6451 40  0000 C CNN
-F 2 "~" V 5980 6450 30  0000 C CNN
-F 3 "~" H 6050 6450 30  0000 C CNN
-	1    6050 6450
-	0    -1   -1   0
-$EndComp
-Wire Wire Line
-	5300 6450 5800 6450
-Wire Wire Line
-	6300 6450 6750 6450
 Wire Wire Line
 	6650 6100 6450 6100
@@
 Text Label 6100 1300 2    60   ~ 0
 V+_MON
-$Comp
-L LM324 U?
-U 1 1 52F141D5
-P 9550 5000
-F 0 "U?" H 9600 5200 60  0000 C CNN
-F 1 "LM324" H 9700 4800 50  0000 C CNN
-F 2 "" H 9550 5000 60  0000 C CNN
-F 3 "" H 9550 5000 60  0000 C CNN
-	1    9550 5000
-	1    0    0    -1
-$EndComp
-$Comp
-L +12V #PWR?
-U 1 1 52F141F1
-P 9450 5500
-F 0 "#PWR?" H 9450 5450 20  0001 C CNN
-F 1 "+12V" H 9450 5600 30  0000 C CNN
-F 2 "" H 9450 5500 60  0000 C CNN
-F 3 "" H 9450 5500 60  0000 C CNN
-	1    9450 5500
-	-1   0    0    1
-$EndComp
-$Comp
-L -12V #PWR?
-U 1 1 52F141F7
-P 9450 4550
-F 0 "#PWR?" H 9450 4680 20  0001 C CNN
-F 1 "-12V" H 9450 4650 30  0000 C CNN
-F 2 "" H 9450 4550 60  0000 C CNN
-F 3 "" H 9450 4550 60  0000 C CNN
-	1    9450 4550
-	1    0    0    -1
-$EndComp
-Wire Wire Line
-	9450 5500 9450 5400
-Wire Wire Line
-	9450 4600 9450 4550
 Wire Wire Line
 	7700 4850 6650 4850
 Connection ~ 6650 4850
-$Comp
-L LM324 U?
-U 1 1 52F14427
-P 9550 6350
-F 0 "U?" H 9600 6550 60  0000 C CNN
-F 1 "LM324" H 9700 6150 50  0000 C CNN
-F 2 "" H 9550 6350 60  0000 C CNN
-F 3 "" H 9550 6350 60  0000 C CNN
-	1    9550 6350
-	1    0    0    -1
-$EndComp
-$Comp
-L +12V #PWR?
-U 1 1 52F1442D
-P 9450 5850
-F 0 "#PWR?" H 9450 5800 20  0001 C CNN
-F 1 "+12V" H 9450 5950 30  0000 C CNN
-F 2 "" H 9450 5850 60  0000 C CNN
-F 3 "" H 9450 5850 60  0000 C CNN
-	1    9450 5850
-	-1   0    0    -1
-$EndComp
-$Comp
-L -12V #PWR?
-U 1 1 52F14433
-P 9450 6800
-F 0 "#PWR?" H 9450 6930 20  0001 C CNN
-F 1 "-12V" H 9450 6900 30  0000 C CNN
-F 2 "" H 9450 6800 60  0000 C CNN
-F 3 "" H 9450 6800 60  0000 C CNN
-	1    9450 6800
-	1    0    0    1
-$EndComp
-Wire Wire Line
-	9450 5850 9450 5950
-Wire Wire Line
-	9450 6750 9450 6800
 Wire Wire Line
 	10400 3550 7700 3550
@@
 Wire Wire Line
 	8800 2700 8800 3400
-Wire Wire Line
-	10250 5000 10050 5000
-Wire Wire Line
-	10250 6350 10050 6350
-Wire Wire Line
-	9050 5100 8850 5100
-Wire Wire Line
-	8850 5100 8850 5650
-Wire Wire Line
-	8850 5650 10150 5650
-Wire Wire Line
-	10150 5650 10150 5000
-Connection ~ 10150 5000
-Wire Wire Line
-	9050 6450 8850 6450
-Wire Wire Line
-	8850 6450 8850 7000
-Wire Wire Line
-	8850 7000 10150 7000
-Wire Wire Line
-	10150 7000 10150 6350
-Connection ~ 10150 6350
-Wire Wire Line
-	8550 6250 9050 6250
-Wire Wire Line
-	9050 4900 8550 4900
-Text Label 8950 4900 2    60   ~ 0
-V+_MON
-Text Label 8950 6250 2    60   ~ 0
-V-_MON
 $Comp
 L RVAR R?
@@
 	1    0    0    -1
 $EndComp
+Wire Wire Line
+	6700 900  5350 900
+Wire Wire Line
+	6750 6450 5300 6450
 $EndSCHEMATC

Commit message: Nach Einfuegen Relay-Modul
Parts:
- gave numbers to parts that had none: 15
Changed lines of the file:
@@
 Sheet 8 9
 Title ""
-Date "14 feb 2014"
+Date "17 feb 2014"
 Rev ""
 Comp ""
@@
 $EndDescr
 $Comp
-L +3,3V #PWR?
+L +3,3V #PWR51
 U 1 1 52F11723
 P 9600 2650
-F 0 "#PWR?" H 9600 2610 30  0001 C CNN
+F 0 "#PWR51" H 9600 2610 30  0001 C CNN
 F 1 "+3,3V" H 9600 2760 30  0000 C CNN
 F 2 "" H 9600 2650 60  0000 C CNN
@@
 $EndComp
 $Comp
-L +5V #PWR?
+L +5V #PWR52
 U 1 1 52F1176F
 P 9800 2650
-F 0 "#PWR?" H 9800 2740 20  0001 C CNN
+F 0 "#PWR52" H 9800 2740 20  0001 C CNN
 F 1 "+5V" H 9800 2740 30  0000 C CNN
 F 2 "" H 9800 2650 60  0000 C CNN
@@
 $EndComp
 $Comp
-L -12V #PWR?
+L -12V #PWR45
 U 1 1 52F117B8
 P 4100 4550
-F 0 "#PWR?" H 4100 4680 20  0001 C CNN
+F 0 "#PWR45" H 4100 4680 20  0001 C CNN
 F 1 "-12V" H 4100 4650 30  0000 C CNN
 F 2 "" H 4100 4550 60  0000 C CNN
@@
 $EndComp
 $Comp
-L +12V #PWR?
+L +12V #PWR44
 U 1 1 52F117C0
 P 4100 2750
-F 0 "#PWR?" H 4100 2700 20  0001 C CNN
+F 0 "#PWR44" H 4100 2700 20  0001 C CNN
 F 1 "+12V" H 4100 2850 30  0000 C CNN
 F 2 "" H 4100 2750 60  0000 C CNN
@@
 $EndComp
 $Comp
-L LM317S U?
+L LM317S U10
 U 1 1 52F117EB
 P 4900 6400
-F 0 "U?" H 4700 6600 40  0000 C CNN
+F 0 "U10" H 4700 6600 40  0000 C CNN
 F 1 "LM317S" H 4900 6600 40  0000 L CNN
 F 2 "TO-263" H 4900 6500 30  0000 C CIN
@@
 	4100 4200 4100 4550
 $Comp
-L JUMPER JP?
+L JUMPER JP2
 U 1 1 52F11819
 P 4850 2750
-F 0 "JP?" H 4850 2900 60  0000 C CNN
+F 0 "JP2" H 4850 2900 60  0000 C CNN
 F 1 "JUMPER" H 4850 2670 40  0000 C CNN
 F 2 "~" H 4850 2750 60  0000 C CNN
@@
 $EndComp
 $Comp
-L JUMPER JP?
+L JUMPER JP3
 U 1 1 52F11826
 P 4850 4700
-F 0 "JP?" H 4850 4850 60  0000 C CNN
+F 0 "JP3" H 4850 4850 60  0000 C CNN
 F 1 "JUMPER" H 4850 4620 40  0000 C CNN
 F 2 "~" H 4850 4700 60  0000 C CNN
@@
 	5550 3100 5250 3100
 $Comp
-L AGND #PWR?
+L AGND #PWR43
 U 1 1 52F1185D
 P 3800 3850
-F 0 "#PWR?" H 3800 3850 40  0001 C CNN
+F 0 "#PWR43" H 3800 3850 40  0001 C CNN
 F 1 "AGND" H 3800 3780 50  0000 C CNN
 F 2 "" H 3800 3850 60  0000 C CNN
@@
 $EndComp
 $Comp
-L GND #PWR?
+L GND #PWR42
 U 1 1 52F1186C
 P 3000 3850
-F 0 "#PWR?" H 3000 3850 30  0001 C CNN
+F 0 "#PWR42" H 3000 3850 30  0001 C CNN
 F 1 "GND" H 3000 3780 30  0001 C CNN
 F 2 "" H 3000 3850 60  0000 C CNN
@@
 $EndComp
 $Comp
-L JUMPER JP?
+L JUMPER JP1
 U 1 1 52F11879
 P 3400 3550
-F 0 "JP?" H 3400 3700 60  0000 C CNN
+F 0 "JP1" H 3400 3700 60  0000 C CNN
 F 1 "JUMPER" H 3400 3470 40  0000 C CNN
 F 2 "~" H 3400 3550 60  0000 C CNN
@@
 	3800 3550 3700 3550
 $Comp
-L AGND #PWR?
+L AGND #PWR46
 U 1 1 52F118D3
 P 4250 3750
-F 0 "#PWR?" H 4250 3750 40  0001 C CNN
+F 0 "#PWR46" H 4250 3750 40  0001 C CNN
 F 1 "AGND" H 4250 3680 50  0000 C CNN
 F 2 "" H 4250 3750 60  0000 C CNN
@@
 Connection ~ 4850 3600
 $Comp
-L FE_V+ #PWR?
+L FE_V+ #PWR48
 U 1 1 52F119E9
 P 5550 2650
-F 0 "#PWR?" H 5550 2750 30  0001 C CNN
+F 0 "#PWR48" H 5550 2750 30  0001 C CNN
 F 1 "FE_V+" H 5550 2750 30  0000 C CNN
 F 2 "" H 5550 2650 60  0000 C CNN
@@
 Connection ~ 5550 2750
 $Comp
-L FE_V- #PWR?
+L FE_V- #PWR50
 U 1 1 52F11A11
 P 5600 4800
-F 0 "#PWR?" H 5600 5000 40  0001 C CNN
+F 0 "#PWR50" H 5600 5000 40  0001 C CNN
 F 1 "FE_V-" H 5600 4950 40  0000 C CNN
 F 2 "" H 5600 4800 60  0000 C CNN
@@
 Connection ~ 5600 4700
 $Comp
-L 7805 U?
+L 7805 U8
 U 1 1 52F11ABB
 P 4850 3150
-F 0 "U?" H 5000 2954 60  0000 C CNN
+F 0 "U8" H 5000 2954 60  0000 C CNN
 F 1 "7805" H 4850 3350 60  0000 C CNN
 F 2 "" H 4850 3150 60  0000 C CNN
@@
 $EndComp
 $Comp
-L 7805 U?
+L 7805 U9
 U 1 1 52F11AC8
 P 4850 4150
-F 0 "U?" H 5000 3954 60  0000 C CNN
+F 0 "U9" H 5000 3954 60  0000 C CNN
 F 1 "7805" H 4850 4350 60  0000 C CNN
 F 2 "" H 4850 4150 60  0000 C CNN
@@
 Connection ~ 4400 4700
 $Comp
-L R R?
+L R R18
 U 1 1 52F11B73
 P 5550 5450
-F 0 "R?" V 5630 5450 40  0000 C CNN
+F 0 "R18" V 5630 5450 40  0000 C CNN
 F 1 "R" V 5557 5451 40  0000 C CNN
 F 2 "~" V 5480 5450 30  0000 C CNN
@@
 $EndComp
 $Comp
-L AGND #PWR?
+L AGND #PWR47
 U 1 1 52F11B95
 P 5150 5250
-F 0 "#PWR?" H 5150 5250 40  0001 C CNN
+F 0 "#PWR47" H 5150 5250 40  0001 C CNN
 F 1 "AGND" H 5150 5180 50  0000 C CNN
 F 2 "" H 5150 5250 60  0000 C CNN
@@
 	4400 6450 4500 6450
 $Comp
-L LM317S U?
+L LM317S U11
 U 1 1 52F137FA
 P 4950 950
-F 0 "U?" H 4750 1150 40  0000 C CNN
+F 0 "U11" H 4750 1150 40  0000 C CNN
 F 1 "LM317S" H 4950 1150 40  0000 L CNN
 F 2 "TO-263" H 4950 1050 30  0000 C CIN
@@
 $EndComp
 $Comp
-L FE_V- #PWR?
+L FE_V- #PWR53
 U 1 1 52F13800
 P 10800 3750
-F 0 "#PWR?" H 10800 3950 40  0001 C CNN
+F 0 "#PWR53" H 10800 3950 40  0001 C CNN
 F 1 "FE_V-" H 10800 3900 40  0000 C CNN
 F 2 "" H 10800 3750 60  0000 C CNN
@@
 $EndComp
 $Comp
-L R R?
+L R R21
 U 1 1 52F13806
 P 5600 1900
-F 0 "R?" V 5680 1900 40  0000 C CNN
+F 0 "R21" V 5680 1900 40  0000 C CNN
 F 1 "R" V 5607 1901 40  0000 C CNN
 F 2 "~" V 5530 1900 30  0000 C CNN
@@
 $EndComp
 $Comp
-L AGND #PWR?
+L AGND #PWR49
 U 1 1 52F13812
 P 5600 2200
-F 0 "#PWR?" H 5600 2200 40  0001 C CNN
+F 0 "#PWR49" H 5600 2200 40  0001 C CNN
 F 1 "AGND" H 5600 2130 50  0000 C CNN
 F 2 "" H 5600 2200 60  0000 C CNN
@@
 Connection ~ 5600 900
 $Comp
-L R R?
+L R R22
 U 1 1 52F13964
 P 6650 2400
-F 0 "R?" V 6730 2400 40  0000 C CNN
+F 0 "R22" V 6730 2400 40  0000 C CNN
 F 1 "R" V 6657 2401 40  0000 C CNN
 F 2 "~" V 6580 2400 30  0000 C CNN
@@
 $EndComp
 $Comp
-L R R?
+L R R23
 U 1 1 52F1396A
 P 6650 3000
-F 0 "R?" V 6730 3000 40  0000 C CNN
+F 0 "R23" V 6730 3000 40  0000 C CNN
 F 1 "R" V 6657 3001 40  0000 C CNN
 F 2 "~" V 6580 3000 30  0000 C CNN
@@
 Connection ~ 4850 3550
 $Comp
-L R R?
+L R R24
 U 1 1 52F13A0F
 P 6650 4500
-F 0 "R?" V 6730 4500 40  0000 C CNN
+F 0 "R24" V 6730 4500 40  0000 C CNN
 F 1 "R" V 6657 4501 40  0000 C CNN
 F 2 "~" V 6580 4500 30  0000 C CNN
@@
 $EndComp
 $Comp
-L R R?
+L R R25
 U 1 1 52F13A15
 P 6650 5200
-F 0 "R?" V 6730 5200 40  0000 C CNN
+F 0 "R25" V 6730 5200 40  0000 C CNN
 F 1 "R" V 6657 5201 40  0000 C CNN
 F 2 "~" V 6580 5200 30  0000 C CNN
@@
 	8800 2700 8800 3400
 $Comp
-L RVAR R?
+L RVAR R19
 U 1 1 52F14806
 P 5550 6100
-F 0 "R?" V 5630 6050 50  0000 C CNN
+F 0 "R19" V 5630 6050 50  0000 C CNN
 F 1 "RVAR" V 5470 6160 50  0000 C CNN
 F 2 "~" H 5550 6100 60  0000 C CNN
@@
 $EndComp
 $Comp
-L RVAR R?
+L RVAR R20
 U 1 1 52F1481D
 P 5600 1250
-F 0 "R?" V 5680 1200 50  0000 C CNN
+F 0 "R20" V 5680 1200 50  0000 C CNN
 F 1 "RVAR" V 5520 1310 50  0000 C CNN
 F 2 "~" H 5600 1250 60  0000 C CNN

Commit message: Am Ende der 5. Woche.
Parts:
- removed JP2, JP3: JUMPER, ~, symbol JUMPER
- removed R19: RVAR, ~, symbol RVAR
- removed U10: LM317S, TO-263, symbol LM317S
- removed U8, U9: 7805, symbol 7805
- added C14, C15, C16, C17, C18, C19, C20, C21, C22, C23, C24, C25: C, ~, symbol C
- added D10, D12, D13, D14, D15, D7, D8, D9: MMBD914-7-F, ~, symbol DIODE
- added R19, R52, R53: R, ~, symbol R
- added R54: 715, ~, symbol R
- added R55: 5k, ~, symbol RVAR
- added U7: LM317S, TO-263, symbol LM317S
- added U8, U9: LM337T, TO-220, symbol LM337T
- R20: value RVAR -> 5k
- R21: value R -> 715
Connections:
- net labels removed: V-_MON
- wire segments 61 -> 108
Other:
- note added: "-1.5V to -10V Output"
- note added: "-10V Output\n"
- note added: "1.5 - 10V Output"
- note added: "10V Output\n"
- moved on the sheet: JP1, R20, R21, R22, R25, U11
