File: Terminal_Block.sch (KiCad schematic (older format))
At the start: 0 parts

Commit message: Am Ende der 5. Woche.
Parts:
- added P4: 12 Pin Terminal Block, symbol CONN_12
- added P5: 3 Pin TB, symbol CONN_3
Connections:
- net +3.3V: now also P4.1 (P1)
- net +5V: now also P4.2 (P2)
- net FAN_OUT+: now also P4.8 (P8)
- net FAN_OUT-: now also P4.9 (P9)
- net GND: now also P4.3 (P3)
- net LED_STRING+: now also P4.6 (P6)
- net LED_STRING-: now also P4.7 (P7)
- net RELAY_COM: now also P5.2 (PM)
- net RELAY_NC: now also P5.3 (P3)
- net RELAY_NO: now also P5.1 (P1)
- net TACH_IN: now also P4.10 (P10)
- net TC_IN+: now also P4.11 (P11)
- net TC_IN-: now also P4.12 (P12)
- net V+_ADJ: now also P4.4 (P4)
- net V-_ADJ: now also P4.5 (P5)
Changed lines of the file:
@@
 $Descr A4 11693 8268
 encoding utf-8
-Sheet 7 9
+Sheet 6 9
 Title ""
-Date "17 feb 2014"
+Date "22 feb 2014"
 Rev ""
 Comp ""
@@
 Comment4 ""
 $EndDescr
-Text HLabel 1850 2850 0    60   Input ~ 0
+Text HLabel 1650 1550 0    60   Input ~ 0
 V+_ADJ
-Text HLabel 1850 3100 0    60   Input ~ 0
+Text HLabel 1650 1650 0    60   Input ~ 0
 V-_ADJ
-Text HLabel 1850 3350 0    60   Output ~ 0
+Text HLabel 1650 2100 0    60   Output ~ 0
 FAN_OUT+
-Text HLabel 1850 3600 0    60   Output ~ 0
+Text HLabel 1650 2200 0    60   Output ~ 0
 FAN_OUT-
-Text HLabel 1850 3800 0    60   Input ~ 0
+Text HLabel 1650 2450 0    60   Input ~ 0
 TACH_IN
-Text HLabel 1850 4050 0    60   Output ~ 0
+Text HLabel 1650 1800 0    60   Output ~ 0
 LED_STRING+
-Text HLabel 1850 4250 0    60   Output ~ 0
+Text HLabel 1650 1900 0    60   Output ~ 0
 LED_STRING-
-Text HLabel 1850 4450 0    60   Input ~ 0
+Text HLabel 1650 2750 0    60   Input ~ 0
 TC_IN+
-Text HLabel 1850 4600 0    60   Input ~ 0
+Text HLabel 1650 2850 0    60   Input ~ 0
 TC_IN-
-Text HLabel 1800 5450 0    60   BiDi ~ 0
+Text HLabel 1650 4200 0    60   BiDi ~ 0
 RELAY_COM
-Text HLabel 1800 5600 0    60   BiDi ~ 0
+Text HLabel 1650 4500 0    60   BiDi ~ 0
 RELAY_NC
-Text HLabel 1800 5750 0    60   BiDi ~ 0
+Text HLabel 1650 3900 0    60   BiDi ~ 0
 RELAY_NO
 $Comp
-L +3.3V #PWR33
+L +3.3V #PWR038
 U 1 1 52F2C1C6
-P 1650 1350
-F 0 "#PWR33" H 1650 1310 30  0001 C CNN
-F 1 "+3.3V" H 1650 1460 30  0000 C CNN
-F 2 "" H 1650 1350 60  0000 C CNN
-F 3 "" H 1650 1350 60  0000 C CNN
-	1    1650 1350
+P 1650 950
+F 0 "#PWR038" H 1650 910 30  0001 C CNN
+F 1 "+3.3V" H 1650 1060 30  0000 C CNN
+F 2 "" H 1650 950 60  0000 C CNN
+F 3 "" H 1650 950 60  0000 C CNN
+	1    1650 950
 	1    0    0    -1
 $EndComp
 $Comp
-L +5V #PWR34
+L +5V #PWR039
 U 1 1 52F2C1D5
-P 1650 1550
-F 0 "#PWR34" H 1650 1640 20  0001 C CNN
-F 1 "+5V" H 1650 1640 30  0000 C CNN
-F 2 "" H 1650 1550 60  0000 C CNN
-F 3 "" H 1650 1550 60  0000 C CNN
-	1    1650 1550
+P 1650 1150
+F 0 "#PWR039" H 1650 1240 20  0001 C CNN
+F 1 "+5V" H 1650 1240 30  0000 C CNN
+F 2 "" H 1650 1150 60  0000 C CNN
+F 3 "" H 1650 1150 60  0000 C CNN
+	1    1650 1150
 	1    0    0    -1
 $EndComp
 $Comp
-L GND #PWR35
+L GND #PWR040
 U 1 1 52F2C1E4
-P 1650 1750
-F 0 "#PWR35" H 1650 1750 30  0001 C CNN
-F 1 "GND" H 1650 1680 30  0001 C CNN
-F 2 "" H 1650 1750 60  0000 C CNN
-F 3 "" H 1650 1750 60  0000 C CNN
-	1    1650 1750
+P 1650 1400
+F 0 "#PWR040" H 1650 1400 30  0001 C CNN
+F 1 "GND" H 1650 1330 30  0001 C CNN
+F 2 "" H 1650 1400 60  0000 C CNN
+F 3 "" H 1650 1400 60  0000 C CNN
+	1    1650 1400
 	1    0    0    -1
 $EndComp
+$Comp
+L CONN_12 P4
+U 1 1 530487DD
+P 4550 1700
+F 0 "P4" V 4500 1700 60  0000 C CNN
+F 1 "12 Pin Terminal Block" V 4600 1700 60  0000 C CNN
+F 2 "" H 4550 1700 60  0000 C CNN
+F 3 "" H 4550 1700 60  0000 C CNN
+F 4 "On Shore" H 4550 1700 60  0001 C CNN "MFG Name"
+F 5 "OSTTE120104" H 4550 1700 60  0001 C CNN "MFG Part Number"
+	1    4550 1700
+	1    0    0    -1
+$EndComp
+Wire Wire Line
+	4200 1350 1650 1350
+Wire Wire Line
+	1650 1350 1650 1400
+Wire Wire Line
+	4200 1250 1650 1250
+Wire Wire Line
+	1650 1250 1650 1150
+Wire Wire Line
+	4200 1150 1850 1150
+Wire Wire Line
+	1850 1150 1850 1000
+Wire Wire Line
+	1850 1000 1650 1000
+Wire Wire Line
+	1650 1000 1650 950
+Wire Wire Line
+	4200 1450 1850 1450
+Wire Wire Line
+	1850 1450 1850 1550
+Wire Wire Line
+	1850 1550 1650 1550
+Wire Wire Line
+	4200 1550 1950 1550
+Wire Wire Line
+	1950 1550 1950 1650
+Wire Wire Line
+	1950 1650 1650 1650
+Wire Wire Line
+	1650 1800 2050 1800
+Wire Wire Line
+	2050 1800 2050 1650
+Wire Wire Line
+	2050 1650 4200 1650
+Wire Wire Line
+	4200 1750 2150 1750
+Wire Wire Line
+	2150 1750 2150 1900
+Wire Wire Line
+	2150 1900 1650 1900
+Wire Wire Line
+	1650 2100 2250 2100
+Wire Wire Line
+	2250 2100 2250 1850
+Wire Wire Line
+	2250 1850 4200 1850
+Wire Wire Line
+	4200 1950 2350 1950
+Wire Wire Line
+	2350 1950 2350 2200
+Wire Wire Line
+	2350 2200 1650 2200
+Wire Wire Line
+	1650 2450 2450 2450
+Wire Wire Line
+	2450 2450 2450 2050
+Wire Wire Line
+	2450 2050 4200 2050
+Wire Wire Line
+	4200 2150 2600 2150
+Wire Wire Line
+	2600 2150 2600 2750
+Wire Wire Line
+	2600 2750 1650 2750
+Wire Wire Line
+	1650 2850 2800 2850
+Wire Wire Line
+	2800 2850 2800 2250
+Wire Wire Line
+	2800 2250 4200 2250
+$Comp
+L CONN_3 P5
+U 1 1 530489C7
+P 2450 4200
+F 0 "P5" V 2400 4200 50  0000 C CNN
+F 1 "3 Pin TB" V 2500 4200 40  0000 C CNN
+F 2 "" H 2450 4200 60  0000 C CNN
+F 3 "" H 2450 4200 60  0000 C CNN
+F 4 "Phoenix" H 2450 4200 60  0001 C CNN "MFG Name"
+F 5 "1935174" H 2450 4200 60  0001 C CNN "MFG Part Number"
+	1    2450 4200
+	1    0    0    -1
+$EndComp
+Wire Wire Line
+	2100 4200 1650 4200
+Wire Wire Line
+	2100 4100 1900 4100
+Wire Wire Line
+	1900 4100 1900 3900
+Wire Wire Line
+	1900 3900 1650 3900
+Wire Wire Line
+	2100 4300 1900 4300
+Wire Wire Line
+	1900 4300 1900 4500
+Wire Wire Line
+	1900 4500 1650 4500
 $EndSCHEMATC
